File: psu_board_small.sch (KiCad schematic (older format))
At the start: 36 parts, among them J1 AC, J2 LED, J3 LED, J4 DC

Commit message: added sch
Parts:
- removed C1, C13, C14, C15, C16, C2: 100n, Capacitor_THT:C_Rect_L7.2mm_W2.5mm_P5.00mm_FKS2_FKP2_MKS2_MKP2, symbol Device:C_Small
- removed R7, R8: 10R, Resistor_THT:R_Axial_DIN0207_L6.3mm_D2.5mm_P10.16mm_Horizontal, symbol Device:R_Small
- added HS1: HSS08-B18-CP, symbol Mechanical:Heatsink
- added HS2: HSC-06, symbol Mechanical:Heatsink
Other:
- moved on the sheet: D2, D3, J1, J2, J3, J4, R10, R11, R12, R9, RV1

Commit message: finished pcb layout
Parts:
- removed HS1: HSS08-B18-CP, symbol Mechanical:Heatsink
- removed HS2: HSC-06, symbol Mechanical:Heatsink
- added C11, C12, C13, C14: 100n, Capacitor_THT:C_Rect_L7.2mm_W2.5mm_P5.00mm_FKS2_FKP2_MKS2_MKP2, symbol Device:C_Small
- added H1, H2, H3, H4: MountingHole, MountingHole:MountingHole_3.2mm_M3_Pad_Via, symbol Mechanical:MountingHole
- added R7, R8: 10R, Resistor_THT:R_Axial_DIN0207_L6.3mm_D2.5mm_P10.16mm_Horizontal, symbol Device:R_Small
- J1: footprint (none) -> TerminalBlock_Phoenix:TerminalBlock_Phoenix_MKDS-1,5-4_1x04_P5.00mm_Horizontal
- J2, J3: footprint (none) -> TerminalBlock_MetzConnect:TerminalBlock_MetzConnect_Type059_RT06302HBWC_1x02_P3.50mm_Horizontal
- J4: footprint (none) -> TerminalBlock_Phoenix:TerminalBlock_Phoenix_MKDS-1,5-6_1x06_P5.00mm_Horizontal
- RV1: footprint (none) -> Varistor:RV_Disc_D15.5mm_W3.9mm_P7.5mm
- renumbered C3 to C1, C12 to C10, C4 to C2, C5 to C3, C6 to C4, C7 to C5, C8 to C6, C9 to C7, C10 to C8, C11 to C9
Connections:
- net GND: now also C11.2, C12.1, C14.1, R7.2
- net OV+: now also C11.1, C13.1
- net OV-: now also C12.2, R8.2
- new net: C13.2, R7.1
- new net: C14.2, R8.1
Other:
- moved on the sheet: D2, D3, J2, J3, J4, R10, R11, R12, R9

Commit message: updated rev2
Parts:
- removed C13, C14: 100n, Capacitor_THT:C_Rect_L7.2mm_W2.5mm_P5.00mm_FKS2_FKP2_MKS2_MKP2, symbol Device:C_Small
- removed J1: AC, TerminalBlock_Phoenix:TerminalBlock_Phoenix_MKDS-1,5-4_1x04_P5.00mm_Horizontal, symbol Connector:Screw_Terminal_01x04
- removed J4: DC, TerminalBlock_Phoenix:TerminalBlock_Phoenix_MKDS-1,5-6_1x06_P5.00mm_Horizontal, symbol Connector:Screw_Terminal_01x06
- removed R3, R4, R5, R6: 0.47R 3W, Resistor_THT:R_Axial_DIN0614_L14.3mm_D5.7mm_P20.32mm_Horizontal, symbol Device:R_Small
- removed R7, R8: 10R, Resistor_THT:R_Axial_DIN0207_L6.3mm_D2.5mm_P10.16mm_Horizontal, symbol Device:R_Small
- added C1, C2: 100n, Capacitor_THT:C_Rect_L7.2mm_W2.5mm_P5.00mm_FKS2_FKP2_MKS2_MKP2, symbol Device:C_Small
- added J1: AC1, local_footprints_lib:Terminal_.25_PCB_TAB_TE_Connectivity_P5.08mm_, symbol Connector:Conn_01x01_Male
- added J10, J9: GND, local_footprints_lib:Terminal_.25_PCB_TAB_TE_Connectivity_P5.08mm_, symbol Connector:Conn_01x01_Male
- added J11, J12: V-, local_footprints_lib:Terminal_.25_PCB_TAB_TE_Connectivity_P5.08mm_, symbol Connector:Conn_01x01_Male
- added J2: GND2, local_footprints_lib:Terminal_.25_PCB_TAB_TE_Connectivity_P5.08mm_, symbol Connector:Conn_01x01_Male
- added J3: GND3, local_footprints_lib:Terminal_.25_PCB_TAB_TE_Connectivity_P5.08mm_, symbol Connector:Conn_01x01_Male
- added J4: AC4, local_footprints_lib:Terminal_.25_PCB_TAB_TE_Connectivity_P5.08mm_, symbol Connector:Conn_01x01_Male
- added J7, J8: V+, local_footprints_lib:Terminal_.25_PCB_TAB_TE_Connectivity_P5.08mm_, symbol Connector:Conn_01x01_Male
- renumbered C6 to C10, C7 to C13, C8 to C14, C1 to C3, C2 to C4, C3 to C5, C4 to C6, C9 to C7, C10 to C8, C5 to C9, J2 to J5, J3 to J6, R9 to R3, R10 to R4, R11 to R5, R12 to R6
Connections:
- net RV+ is gone; now on net V+: C13.1, C3.1, C5.1, C9.1, D1.1 (+)
- net RV- is gone; now on net V-: C10.2, C4.2, C6.2, D1.4 (-), R2.2
- net AC1: now also C1.1, J1.1 (Pin_1)
- net AC4: now also C2.2, J4.1 (Pin_1)
- net GND: now also C1.2, C2.1, J10.1 (Pin_1), J2.1 (Pin_1), J3.1 (Pin_1), J9.1 (Pin_1)
- net OV+ renamed V+
- net V+: now also J7.1 (Pin_1), J8.1 (Pin_1)
- net OV- renamed V-
- net V-: now also J11.1 (Pin_1), J12.1 (Pin_1)
Other:
- moved on the sheet: C10, C13, C14, C7, C8, C9, D1, D2, D3, J5, J6, R1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
